File: Thermal_Shield/Thermal_Shield.kicad_pcb (KiCad board)
At the start: 2 copper layers, 19 parts, among them J1 Screw_Terminal_01x03, J2 Barrel_Jack_Switch, Q1 BC337, Q2 BC337, Q3 BC337, U1 LM35-D, U2 LM311

Commit message: PCB ready to connections
Parts:
- C1: footprint Capacitor_THT:C_Rect_L9.0mm_W2.5mm_P7.50mm_MKT -> Capacitor_THT:C_Rect_L7.2mm_W2.5mm_P5.00mm_FKS2_FKP2_MKS2_MKP2
- Q1, Q2, Q3, U1: footprint Package_TO_SOT_THT:TO-92_Inline -> Package_TO_SOT_THT:TO-92_Inline_Wide
- R1: renamed from R2; footprint Resistor_THT:R_Axial_DIN0516_L15.5mm_D5.0mm_P20.32mm_Horizontal -> Resistor_THT:R_Axial_DIN0309_L9.0mm_D3.2mm_P12.70mm_Horizontal
- R2: renamed from R1; footprint Resistor_THT:R_Axial_DIN0516_L15.5mm_D5.0mm_P20.32mm_Horizontal -> Resistor_THT:R_Axial_DIN0309_L9.0mm_D3.2mm_P12.70mm_Horizontal
- R3: renamed from R4; footprint Resistor_THT:R_Axial_DIN0516_L15.5mm_D5.0mm_P20.32mm_Horizontal -> Resistor_THT:R_Axial_DIN0309_L9.0mm_D3.2mm_P12.70mm_Horizontal
- R4: renamed from R8; footprint Resistor_THT:R_Axial_DIN0516_L15.5mm_D5.0mm_P20.32mm_Horizontal -> Resistor_THT:R_Axial_DIN0309_L9.0mm_D3.2mm_P12.70mm_Horizontal
- R5: renamed from R7; footprint Resistor_THT:R_Axial_DIN0516_L15.5mm_D5.0mm_P20.32mm_Horizontal -> Resistor_THT:R_Axial_DIN0309_L9.0mm_D3.2mm_P12.70mm_Horizontal
- R6: footprint Resistor_THT:R_Axial_DIN0516_L15.5mm_D5.0mm_P20.32mm_Horizontal -> Resistor_THT:R_Axial_DIN0309_L9.0mm_D3.2mm_P12.70mm_Horizontal
- R7: renamed from R5; footprint Resistor_THT:R_Axial_DIN0516_L15.5mm_D5.0mm_P20.32mm_Horizontal -> Resistor_THT:R_Axial_DIN0309_L9.0mm_D3.2mm_P12.70mm_Horizontal
- R8: renamed from R3; footprint Resistor_THT:R_Box_L26.0mm_W5.0mm_P20.00mm -> Resistor_THT:R_Axial_DIN0309_L9.0mm_D3.2mm_P20.32mm_Horizontal
- U2: footprint Package_DIP:CERDIP-8_W7.62mm_SideBrazed -> Package_DIP:DIP-8_W7.62mm
- moved R7 92.5 mm to (45.0, 57.5)
- moved Q3 82.5 mm to (55.2, 74.0)
- moved Q2 79.6 mm to (59.8, 52.5), turned to 180 degrees
- moved R5 67.4 mm to (26.8, 46.8)
- moved Q1 64.4 mm to (42.0, 49.2)
- moved J2 62.5 mm to (59.8, 46.5)
- moved U1 59.2 mm to (56.8, 61.0)
- moved R8 58.3 mm to (63.8, 74.2)
- moved C1 56.0 mm to (45.2, 73.4), turned to 0 degrees
- moved U2 50.1 mm to (45.2, 62.4)
- moved R6 45.7 mm to (50.5, 37.6), turned to -90 degrees
- moved R4 33.8 mm to (41.0, 67.8)
- moved J1 25.5 mm to (30.2, 74.5)
- moved D1 20.0 mm to (30.5, 40.0)
- moved D2 19.6 mm to (37.5, 40.0)
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Connections:
- C1 pad 1: Net-(Q3-E) -> Net-(Q3-C)
- J2 pad 1: GND -> IN_12
- J2 pad 2: IN_12 -> GND
- Q3 pad 1: IN_12 -> Net-(Q3-C)
- Q3 pad 3: Net-(Q3-E) -> IN_12
- U2 pad 7: Net-(Q3-E) -> Net-(Q3-C)
- U2 pad 8: Net-(Q3-E) -> Net-(Q3-C)

Commit message: Connections
Parts:
- U1: value LM35-D -> LM35-LP
- moved R7 19.9 mm to (58.0, 57.5), turned to 180 degrees
- moved C1 5.00 mm to (50.2, 73.4), turned to 180 degrees
- moved R4 4.68 mm to (41.0, 55.1), turned to -90 degrees
- moved J1 1.25 mm to (29.0, 74.5)
- moved J2 0.50 mm to (59.8, 46.0)
- moved Q3 0.16 mm to (55.2, 74.2)
- renumbered R7 to R4, R4 to R7
Connections:
- C1 pad 2: Net-(U2-GND) -> GND
- J1 pad 1: PMW -> GND
- J1 pad 3: GND -> PWM
- Q1 pad 1: GND -> Net-(Q1-C)
- Q1 pad 3: Net-(Q1-E) -> GND
- Q2 pad 2: Net-(Q1-E) -> Net-(Q1-C)
- R3 pad 1: Net-(Q1-E) -> Net-(Q1-C)
- R4 pad 1: Net-(U1-+V_{S}) -> Net-(Q3-C)
- U1 pad 1: V_T -> Net-(Q3-C)
- U1 pad 2: unconnected-(U1-NC-Pad2) -> V_T
- U1 pad 3: unconnected-(U1-NC-Pad3) -> GND
Routing:
- net GND: track 0.00 -> 156.0 mm
- net IN_12: track 0.00 -> 64.2 mm
- net V_T: track 0.00 -> 52.4 mm
- net Net-(U2-+): track 0.00 -> 50.6 mm
- net Net-(Q1-C): track 0.00 -> 41.4 mm
- net Net-(Q3-C): track 0.00 -> 41.2 mm
- net Net-(U2-GND): track 0.00 -> 27.4 mm
- net Net-(D2-A): track 0.00 -> 17.4 mm
- net Net-(Q1-B): track 0.00 -> 16.9 mm
- net Net-(D1-A): track 0.00 -> 13.7 mm
- net PWM: track 0.00 -> 12.8 mm
- net Net-(D3-A): track 0.00 -> 12.6 mm
- net Net-(Q2-C): track 0.00 -> 4.52 mm
Other:
- board outline added: 43.8 x 45 mm
- board text added: "Alarm"
- board text added: "Alim"
- board text added: "GND"
- board text added: "PWM"
- board text added: "Sistema Termico"
- board text added: "V_T"
