File: Thermal_Shield/Thermal_Shield.kicad_sch (KiCad schematic)
At the start: 19 parts, among them J1 Screw_Terminal_01x03, J2 Barrel_Jack_Switch, Q1 BC337, Q2 BC337, Q3 BC337, U1 LM35-D, U2 LM311

Commit message: PCB ready to connections
Parts:
- C1: footprint Capacitor_THT:C_Rect_L9.0mm_W2.5mm_P7.50mm_MKT -> Capacitor_THT:C_Rect_L7.2mm_W2.5mm_P5.00mm_FKS2_FKP2_MKS2_MKP2
- Q1, Q2, Q3, U1: footprint Package_TO_SOT_THT:TO-92_Inline -> Package_TO_SOT_THT:TO-92_Inline_Wide
- R1: renamed from R2; footprint Resistor_THT:R_Axial_DIN0516_L15.5mm_D5.0mm_P20.32mm_Horizontal -> Resistor_THT:R_Axial_DIN0309_L9.0mm_D3.2mm_P12.70mm_Horizontal
- R2: renamed from R1; footprint Resistor_THT:R_Axial_DIN0516_L15.5mm_D5.0mm_P20.32mm_Horizontal -> Resistor_THT:R_Axial_DIN0309_L9.0mm_D3.2mm_P12.70mm_Horizontal
- R3: renamed from R4; footprint Resistor_THT:R_Axial_DIN0516_L15.5mm_D5.0mm_P20.32mm_Horizontal -> Resistor_THT:R_Axial_DIN0309_L9.0mm_D3.2mm_P12.70mm_Horizontal
- R4: renamed from R8; footprint Resistor_THT:R_Axial_DIN0516_L15.5mm_D5.0mm_P20.32mm_Horizontal -> Resistor_THT:R_Axial_DIN0309_L9.0mm_D3.2mm_P12.70mm_Horizontal
- R5: renamed from R7; footprint Resistor_THT:R_Axial_DIN0516_L15.5mm_D5.0mm_P20.32mm_Horizontal -> Resistor_THT:R_Axial_DIN0309_L9.0mm_D3.2mm_P12.70mm_Horizontal
- R6: footprint Resistor_THT:R_Axial_DIN0516_L15.5mm_D5.0mm_P20.32mm_Horizontal -> Resistor_THT:R_Axial_DIN0309_L9.0mm_D3.2mm_P12.70mm_Horizontal
- R7: renamed from R5; footprint Resistor_THT:R_Axial_DIN0516_L15.5mm_D5.0mm_P20.32mm_Horizontal -> Resistor_THT:R_Axial_DIN0309_L9.0mm_D3.2mm_P12.70mm_Horizontal
- R8: renamed from R3; footprint Resistor_THT:R_Box_L26.0mm_W5.0mm_P20.00mm -> Resistor_THT:R_Axial_DIN0309_L9.0mm_D3.2mm_P20.32mm_Horizontal
- U2: footprint Package_DIP:CERDIP-8_W7.62mm_SideBrazed -> Package_DIP:DIP-8_W7.62mm
Connections:
- net GND: now also J2.2; no longer J2.1
- net IN_12: now also J2.1, Q3.3 (E); no longer J2.2, Q3.1 (C)
- net at C1.1, U2.7, U2.8 (V+): now also Q3.1 (C); no longer Q3.3 (E)
Other:
- moved on the sheet: Q3
Changed lines of the file:
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@@
+	(wire
+		(pts
+			(xy 113.03 33.02) (xy 113.03 36.83)
+		)
+		(stroke
+			(width 0)
+			(type default)
+		)
+	)
 	(wire
 		(pts
@@
 	(wire
 		(pts
-			(xy 113.03 33.02) (xy 113.03 36.83)
+			(xy 118.11 33.02) (xy 118.11 36.83)
 		)
 		(stroke
@@
 		(pts
 			(xy 43.18 100.33) (xy 43.18 102.87)
-		)
-		(stroke
-			(width 0)
-			(type default)
-		)
-	)
-	(wire
-		(pts
-			(xy 118.11 33.02) (xy 118.11 36.83)
 		)
 		(stroke
@@
 	(global_label "GND"
 		(shape input)
-		(at 118.11 36.83 270)
+		(at 113.03 36.83 270)
 		(fields_autoplaced yes)
 		(effects
@@
 		)
 		(property "Intersheetrefs" "${INTERSHEET_REFS}"
-			(at 118.11 43.6857 90)
+			(at 113.03 43.6857 90)
 			(effects
 				(font
@@
 	(global_label "IN_12"
 		(shape input)
-		(at 113.03 36.83 270)
+		(at 118.11 36.83 270)
 		(fields_autoplaced yes)
 		(effects
@@
 		)
 		(property "Intersheetrefs" "${INTERSHEET_REFS}"
-			(at 113.03 45.1371 90)
+			(at 118.11 45.1371 90)
 			(effects
 				(font
@@
 		(dnp no)
 		(fields_autoplaced yes)
-		(property "Reference" "R8"
+		(property "Reference" "R4"
 			(at 172.72 93.9799 0)
 			(effects
@@
 			)
 		)
-		(property "Footprint" "Resistor_THT:R_Axial_DIN0516_L15.5mm_D5.0mm_P20.32mm_Horizontal"
+		(property "Footprint" "Resistor_THT:R_Axial_DIN0309_L9.0mm_D3.2mm_P12.70mm_Horizontal"
 			(at 171.958 95.25 90)
 			(effects
@@
 			(project "Thermal_Shield"
 				(path "/86db98c8-2a21-4833-9f48-3f46b4aadc3c"
-					(reference "R8")
+					(reference "R4")
 					(unit 1)
 				)
@@
 		(dnp no)
 		(fields_autoplaced yes)
-		(property "Reference" "R3"
+		(property "Reference" "R8"
 			(at 207.01 113.0299 0)
 			(effects
@@
 			)
 		)
-		(property "Footprint" "Resistor_THT:R_Box_L26.0mm_W5.0mm_P20.00mm"
+		(property "Footprint" "Resistor_THT:R_Axial_DIN0309_L9.0mm_D3.2mm_P20.32mm_Horizontal"
 			(at 202.692 114.3 90)
 			(effects
@@
 			(project ""
 				(path "/86db98c8-2a21-4833-9f48-3f46b4aadc3c"
-					(reference "R3")
+					(reference "R8")
 					(unit 1)
 				)
@@
 			)
 		)
-		(property "Footprint" "Resistor_THT:R_Axial_DIN0516_L15.5mm_D5.0mm_P20.32mm_Horizontal"
+		(property "Footprint" "Resistor_THT:R_Axial_DIN0309_L9.0mm_D3.2mm_P12.70mm_Horizontal"
 			(at 66.548 106.68 90)
 			(effects
@@
 			)
 		)
-		(property "Footprint" "Package_DIP:CERDIP-8_W7.62mm_SideBrazed"
+		(property "Footprint" "Package_DIP:DIP-8_W7.62mm"
 			(at 107.95 102.87 0)
 			(effects
@@
 		(dnp no)
 		(fields_autoplaced yes)
-		(property "Reference" "R2"
+		(property "Reference" "R1"
 			(at 45.72 105.4099 0)
 			(effects
@@
 			)
 		)
-		(property "Footprint" "Resistor_THT:R_Axial_DIN0516_L15.5mm_D5.0mm_P20.32mm_Horizontal"
+		(property "Footprint" "Resistor_THT:R_Axial_DIN0309_L9.0mm_D3.2mm_P12.70mm_Horizontal"
 			(at 44.958 106.68 90)
 			(effects
@@
 			(project "Thermal_Shield"
 				(path "/86db98c8-2a21-4833-9f48-3f46b4aadc3c"
-					(reference "R2")
+					(reference "R1")
 					(unit 1)
 				)
@@
 			)
 		)
-		(property "Footprint" "Package_TO_SOT_THT:TO-92_Inline"
+		(property "Footprint" "Package_TO_SOT_THT:TO-92_Inline_Wide"
 			(at 193.675 124.46 0)
 			(effects
@@
 		(dnp no)
 		(fields_autoplaced yes)
-		(property "Reference" "R1"
+		(property "Reference" "R2"
 			(at 57.15 105.4099 0)
 			(effects
@@
 			)
 		)
-		(property "Footprint" "Resistor_THT:R_Axial_DIN0516_L15.5mm_D5.0mm_P20.32mm_Horizontal"
+		(property "Footprint" "Resistor_THT:R_Axial_DIN0309_L9.0mm_D3.2mm_P12.70mm_Horizontal"
 			(at 56.388 106.68 90)
 			(effects
@@
 			(project "Thermal_Shield"
 				(path "/86db98c8-2a21-4833-9f48-3f46b4aadc3c"
-					(reference "R1")
+					(reference "R2")
 					(unit 1)
 				)
@@
 		(dnp no)
 		(fields_autoplaced yes)
-		(property "Reference" "R7"
+		(property "Reference" "R5"
 			(at 90.17 81.28 90)
 			(effects
@@
 			)
 		)
-		(property "Footprint" "Resistor_THT:R_Axial_DIN0516_L15.5mm_D5.0mm_P20.32mm_Horizontal"
+		(property "Footprint" "Resistor_THT:R_Axial_DIN0309_L9.0mm_D3.2mm_P12.70mm_Horizontal"
 			(at 90.17 85.852 90)
 			(effects
@@
 			(project "Thermal_Shield"
 				(path "/86db98c8-2a21-4833-9f48-3f46b4aadc3c"
-					(reference "R7")
+					(reference "R5")
 					(unit 1)
 				)
@@
 			)
 		)
-		(property "Footprint" "Capacitor_THT:C_Rect_L9.0mm_W2.5mm_P7.50mm_MKT"
+		(property "Footprint" "Capacitor_THT:C_Rect_L7.2mm_W2.5mm_P5.00mm_FKS2_FKP2_MKS2_MKP2"
 			(at 109.22 145.7452 0)
 			(effects
@@
 	(symbol
 		(lib_id "Transistor_BJT:BC337")
-		(at 184.15 133.35 270)
+		(at 184.15 133.35 90)
+		(mirror x)
 		(unit 1)
 		(exclude_from_sim no)
@@
 		(on_board yes)
 		(dnp no)
-		(fields_autoplaced yes)
 		(property "Reference" "Q3"
 			(at 184.15 139.7 90)
@@
 			)
 		)
-		(property "Footprint" "Package_TO_SOT_THT:TO-92_Inline"
-			(at 182.245 138.43 0)
+		(property "Footprint" "Package_TO_SOT_THT:TO-92_Inline_Wide"
+			(at 186.055 138.43 0)
 			(effects
 				(font
@@
 			)
 		)
-		(property "Footprint" "Package_TO_SOT_THT:TO-92_Inline"
+		(property "Footprint" "Package_TO_SOT_THT:TO-92_Inline_Wide"
 			(at 172.085 111.76 0)
 			(effects
@@
 			)
 		)
-		(property "Footprint" "Package_TO_SOT_THT:TO-92_Inline"
+		(property "Footprint" "Package_TO_SOT_THT:TO-92_Inline_Wide"
 			(at 138.43 123.19 0)
 			(effects
@@
 		(dnp no)
 		(fields_autoplaced yes)
-		(property "Reference" "R5"
+		(property "Reference" "R7"
 			(at 140.97 92.7099 0)
 			(effects
@@
 			)
 		)
-		(property "Footprint" "Resistor_THT:R_Axial_DIN0516_L15.5mm_D5.0mm_P20.32mm_Horizontal"
+		(property "Footprint" "Resistor_THT:R_Axial_DIN0309_L9.0mm_D3.2mm_P12.70mm_Horizontal"
 			(at 140.208 93.98 90)
 			(effects
@@
 			(project "Thermal_Shield"
 				(path "/86db98c8-2a21-4833-9f48-3f46b4aadc3c"
-					(reference "R5")
+					(reference "R7")
 					(unit 1)
 				)
@@
 		(dnp no)
 		(fields_autoplaced yes)
-		(property "Reference" "R4"
+		(property "Reference" "R3"
 			(at 198.12 97.7899 0)
 			(effects
@@
 			)
 		)
-		(property "Footprint" "Resistor_THT:R_Axial_DIN0516_L15.5mm_D5.0mm_P20.32mm_Horizontal"
+		(property "Footprint" "Resistor_THT:R_Axial_DIN0309_L9.0mm_D3.2mm_P12.70mm_Horizontal"
 			(at 197.358 99.06 90)
 			(effects
@@
 			(project "Thermal_Shield"
 				(path "/86db98c8-2a21-4833-9f48-3f46b4aadc3c"
-					(reference "R4")
+					(reference "R3")
 					(unit 1)
 				)

Commit message: Connections
Parts:
- removed U1: LM35-D, Package_TO_SOT_THT:TO-92_Inline_Wide, symbol Sensor_Temperature:LM35-D
- added U1: LM35-LP, Package_TO_SOT_THT:TO-92_Inline_Wide, symbol Sensor_Temperature:LM35-LP
- renumbered R7 to R4, R4 to R7
Connections:
- net PMW is gone; now on net GND: J1.1 (Pin_1)
- net GND: now also C1.2, Q1.3 (E), U1.3 (GND); no longer J1.3 (Pin_3), Q1.1 (C)
- net PWM: now also J1.3 (Pin_3)
- net V_T: now also U1.2 (V_{OUT})
- net at R1.1, R7.2, U2.1 (GND): no longer C1.2
- net at C1.1, Q3.1 (C), U2.7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: now also R4.1, U1.1 (+V_{S})
- net at Q2.2 (B), R3.1: now also Q1.1 (C); no longer Q1.3 (E)
Other:
- moved on the sheet: J1, Q1
